File: kicad_project/GuitarAmplifier.kicad_pcb (KiCad board)
At the start: 4 copper layers, 158.5 x 57 mm, 47 parts, among them J1 NMJ6HCD2, U1 TL072CP, U2 TL072CP, U3 LM386

Commit message: Agregando serigrafia trasera
Parts:
- added G***: LOGO, DibujoT.preety:capibara, B.Cu at (164.9, 144.5)
Other:
- board text added: "anthonycalvo50@gmail.com"
- board text added: "rmadrigalmontes@gmail.com"

Commit message: Agregando cambio en conector de switch y modelos 3D de componentes faltantes
Signed-off-by: RoMadrigal <rmadrigalmontes@gmail.com>
Parts:
- removed the G*** at (164.9, 144.5)
- added G***: LOGO, DibujoT:capibara, B.Cu at (163.0, 144.6)
- moved CLEAN / O.D SWITCH 10.3 mm to (219.8, 161.6), turned to 0 degrees
Routing:
- net /OUT_OverD: track 43.3 -> 38.4 mm
- net /OUT_Clean: track 44.3 -> 48.4 mm
Changed lines of the file:
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@@
 			)
 		)
+		(model "${KIPRJMOD}/3Dmodels/TerminalBlock_bornier-2_P5.08mm.step"
+			(offset
+				(xyz 2.54 0 0)
+			)
+			(scale
+				(xyz 1 1 1)
+			)
+			(rotate
+				(xyz 0 0 0)
+			)
+		)
 	)
 	(footprint "TerminalBlock:TerminalBlock_bornier-2_P5.08mm"
@@
 			)
 		)
+		(model "${KIPRJMOD}/3Dmodels/TerminalBlock_bornier-2_P5.08mm.step"
+			(offset
+				(xyz 2.54 0 0)
+			)
+			(scale
+				(xyz 1 1 1)
+			)
+			(rotate
+				(xyz 0 0 0)
+			)
+		)
 	)
 	(footprint "Potentiometer_THT:Potentiometer_Piher_PC-16_Single_Horizontal"
@@
 			)
 		)
+		(model "${KIPRJMOD}/3Dmodels/PotentiometerAssy.STEP"
+			(offset
+				(xyz -4.6 22 11.5)
+			)
+			(scale
+				(xyz 1 1 1)
+			)
+			(rotate
+				(xyz -90 0 -90)
+			)
+		)
 	)
 	(footprint "PCBWayLogo:PCBWayLogo3"
@@
 			)
 		)
+		(model "${KIPRJMOD}/3Dmodels/SJ-63073E--3DModel-STEP-1.STEP"
+			(offset
+				(xyz 6.3 -24.66 6)
+			)
+			(scale
+				(xyz 1 1 1)
+			)
+			(rotate
+				(xyz -90 0 90)
+			)
+		)
 	)
 	(footprint "Capacitor_THT:C_Disc_D7.5mm_W5.0mm_P5.00mm"
@@
 			)
 		)
+		(model "${KIPRJMOD}/3Dmodels/PotentiometerAssy.STEP"
+			(offset
+				(xyz -4.6 22 11.5)
+			)
+			(scale
+				(xyz 1 1 1)
+			)
+			(rotate
+				(xyz -90 0 -90)
+			)
+		)
 	)
 	(footprint "Resistor_THT:R_Axial_DIN0207_L6.3mm_D2.5mm_P7.62mm_Horizontal"
@@
 			)
 		)
+		(model "${KIPRJMOD}/3Dmodels/PotentiometerAssy.STEP"
+			(offset
+				(xyz -4.6 22 11.5)
+			)
+			(scale
+				(xyz 1 1 1)
+			)
+			(rotate
+				(xyz -90 0 -90)
+			)
+		)
 	)
 	(footprint "TerminalBlock:TerminalBlock_bornier-3_P5.08mm"
 		(layer "F.Cu")
-		(at 230.08 161.6 180)
+		(at 219.8 161.6)
 		(descr "simple 3-pin terminal block, pitch 5.08mm, revamped version of bornier3")
 		(tags "terminal block bornier3")
 		(property "Reference" "CLEAN / O.D SWITCH"
-			(at 5.08 -5.8 180)
+			(at 5 5.8 360)
 			(layer "F.SilkS")
 			(effects
@@
 		)
 		(property "Value" "Terminal_01x03"
-			(at 4.93 5.35 180)
+			(at 4.93 5.35 360)
 			(layer "F.Fab")
 			(effects
@@
 		)
 		(property "Footprint" "TerminalBlock:TerminalBlock_bornier-3_P5.08mm"
-			(at 0 0 180)
+			(at 0 0 0)
 			(unlocked yes)
 			(layer "F.Fab")
@@
 		)
 		(property "Datasheet" ""
-			(at 0 0 180)
+			(at 0 0 0)
 			(unlocked yes)
 			(layer "F.Fab")
@@
 		)
 		(property "Description" "Generic screw terminal, single row, 01x03, script generated (kicad-library-utils/schlib/autogen/connector/)"
-			(at 0 0 180)
+			(at 0 0 0)
 			(unlocked yes)
 			(layer "F.Fab")
@@
 		(attr through_hole)
 		(fp_line
-			(start 12.7 3.81)
+			(start -2.54 -3.81)
 			(end 12.7 -3.81)
 			(stroke
@@
 		)
 		(fp_line
-			(start -2.54 3.81)
-			(end 12.7 3.81)
+			(start -2.54 2.54)
+			(end 12.7 2.54)
 			(stroke
 				(width 0.12)
@@
 		)
 		(fp_line
-			(start -2.54 2.54)
-			(end 12.7 2.54)
+			(start -2.54 3.81)
+			(end 12.7 3.81)
 			(stroke
 				(width 0.12)
@@
 		)
 		(fp_line
-			(start -2.54 -3.81)
+			(start 12.7 3.81)
 			(end 12.7 -3.81)
 			(stroke
@@
 		)
 		(fp_line
-			(start 12.88 4)
-			(end 12.88 -4)
+			(start -2.72 -4)
+			(end -2.72 4)
 			(stroke
 				(width 0.05)
@@
 		)
 		(fp_line
-			(start 12.88 4)
-			(end -2.72 4)
+			(start -2.72 -4)
+			(end 12.88 -4)
 			(stroke
 				(width 0.05)
@@
 		)
 		(fp_line
-			(start -2.72 -4)
-			(end 12.88 -4)
+			(start 12.88 4)
+			(end -2.72 4)
 			(stroke
 				(width 0.05)
@@
 		)
 		(fp_line
-			(start -2.72 -4)
-			(end -2.72 4)
+			(start 12.88 4)
+			(end 12.88 -4)
 			(stroke
 				(width 0.05)
@@
 		)
 		(fp_line
-			(start 12.63 3.75)
-			(end -2.47 3.75)
+			(start -2.47 -3.75)
+			(end 12.63 -3.75)
 			(stroke
 				(width 0.1)
@@
 		)
 		(fp_line
-			(start 12.63 -3.75)
-			(end 12.63 3.75)
+			(start -2.47 2.55)
+			(end 12.63 2.55)
 			(stroke
 				(width 0.1)
@@
 		)
 		(fp_line
-			(start -2.47 2.55)
-			(end 12.63 2.55)
+			(start 12.63 -3.75)
+			(end 12.63 3.75)
 			(stroke
 				(width 0.1)
@@
 		)
 		(fp_line
-			(start -2.47 -3.75)
-			(end 12.63 -3.75)
+			(start 12.63 3.75)
+			(end -2.47 3.75)
 			(stroke
 				(width 0.1)
@@
 		)
 		(fp_text user "${REFERENCE}"
-			(at 5.08 0 180)
+			(at 5.08 0 360)
 			(layer "F.Fab")
 			(effects
@@
 		)
 		(pad "1" thru_hole rect
-			(at 0 0 180)
+			(at 0 0)
 			(size 3 3)
 			(drill 1.52)
@@
 		)
 		(pad "2" thru_hole circle
-			(at 5.08 0 180)
+			(at 5.08 0)
 			(size 3 3)
 			(drill 1.52)
@@
 		)
 		(pad "3" thru_hole circle
-			(at 10.16 0 180)
+			(at 10.16 0)
 			(size 3 3)
 			(drill 1.52)
@@
 			)
 		)
+		(model "${KIPRJMOD}/3Dmodels/282836-3--3DModel-STEP-1.STEP"
+			(offset
+				(xyz 5.08 -4 5)
+			)
+			(scale
+				(xyz 1 1 1)
+			)
+			(rotate
+				(xyz -90 0 0)
+			)
+		)
 	)
 	(footprint "Resistor_THT:R_Axial_DIN0207_L6.3mm_D2.5mm_P7.62mm_Horizontal"
@@
 			)
 		)
+		(model "${KIPRJMOD}/3Dmodels/PotentiometerAssy.STEP"
+			(offset
+				(xyz -4.6 22 11.5)
+			)
+			(scale
+				(xyz 1 1 1)
+			)
+			(rotate
+				(xyz -90 0 -90)
+			)
+		)
 	)
 	(footprint "Resistor_THT:R_Axial_DIN0207_L6.3mm_D2.5mm_P7.62mm_Horizontal"
@@
 			)
 		)
+		(model "${KIPRJMOD}/3Dmodels/PotentiometerAssy.STEP"
+			(offset
+				(xyz -4.6 22 11.5)
+			)
+			(scale
+				(xyz 1 1 1)
+			)
+			(rotate
+				(xyz -90 0 -90)
+			)
+		)
 	)
 	(footprint "Package_DIP:DIP-8_W7.62mm"
@@
 		)
 	)
-	(footprint "DibujoT.preety:capibara"
+	(footprint "DibujoT:capibara"
 		(layer "B.Cu")
-		(at 164.927947 144.515962 180)
+		(at 163.027947 144.615962 180)
 		(property "Reference" "G***"
 			(at -0.569703 -0.213741 0)
-			(layer "B.SilkS")
+			(layer "F.SilkS")
 			(hide yes)
 			(effects
@@
 					(thickness 0.3)
 				)
-				(justify mirror)
 			)
 		)
 		(property "Value" "LOGO"
 			(at 0.180297 -0.213741 0)
-			(layer "B.SilkS")
+			(layer "F.SilkS")
 			(hide yes)
 			(effects
@@
 					(thickness 0.3)
 				)
-				(justify mirror)
 			)
 		)
-		(property "Footprint" ""
+		(property "Footprint" "DibujoT:capibara"
 			(at -0.569703 -0.213741 0)
 			(layer "B.Fab")
@@
 	)
 	(gr_text "rmadrigalmontes@gmail.com"
-		(at 258 168.5 0)
+		(at 176.8 168.2 0)
 		(layer "B.SilkS")
 		(effects
 			(font
 				(size 2 3)
-				(thickness 0.1)
+				(thickness 0.375)
+				(bold yes)
 			)
 			(justify left bottom mirror)
@@
 	)
 	(gr_text "anthonycalvo50@gmail.com"
-		(at 165.5 115.5 0)
+		(at 165.5 115.8 0)
 		(layer "B.SilkS")
 		(effects
 			(font
 				(size 2 3)
-				(thickness 0.1)
+				(thickness 0.4)
+				(bold yes)
 			)
 			(justify left bottom mirror)
@@
 	)
 	(segment
-		(start 225 161.6)
-		(end 225 150.5)
+		(start 227 148.5)
+		(end 227 159.48)
 		(width 0.2)
-		(layer "B.Cu")
+		(layer "F.Cu")
 		(net 18)
 	)
 	(segment
-		(start 225 150.5)
-		(end 227 148.5)
+		(start 227 159.48)
+		(end 224.88 161.6)
 		(width 0.2)
-		(layer "B.Cu")
+		(layer "F.Cu")
 		(net 18)
 	)
@@
 	(segment
 		(start 216 141.74)
-		(end 217.149189 141.74)
-		(width 0.3)
-		(layer "F.Cu")
-		(net 20)
-	)
-	(segment
-		(start 216 141.74)
 		(end 220.16 137.58)
 		(width 0.3)
@@
 	)
 	(segment
-		(start 230.08 154.670811)
-		(end 230.08 161.6)
+		(start 219.8 161.6)
+		(end 219.8 145.54)
 		(width 0.3)
 		(layer "F.Cu")
@@
 	)
 	(segment
-		(start 217.149189 141.74)
-		(end 230.08 154.670811)
+		(start 219.8 145.54)
+		(end 216 141.74)
 		(width 0.3)
 		(layer "F.Cu")
@@
 	)
 	(segment
-		(start 216 146.82)
-		(end 216 157.68)
+		(start 199.68 130.5)
+		(end 208.38 139.2)
 		(width 0.3)
 		(layer "F.Cu")
@@
 	)
 	(segment
-		(start 216 157.68)
-		(end 219.92 161.6)
+		(start 194.88 130.5)
+		(end 199.68 130.5)
 		(width 0.3)
 		(layer "F.Cu")
@@
 	)
 	(segment
-		(start 199.68 130.5)
-		(end 208.38 139.2)
+		(start 208.38 139.2)
+		(end 216 146.82)
 		(width 0.3)
 		(layer "F.Cu")
@@
 	)
 	(segment
-		(start 194.88 130.5)
-		(end 199.68 130.5)
+		(start 216 146.82)
+		(end 229.96 160.78)
 		(width 0.3)
-		(layer "F.Cu")
+		(layer "B.Cu")
 		(net 23)
 	)
 	(segment
-		(start 208.38 139.2)
-		(end 216 146.82)
+		(start 229.96 160.78)
+		(end 229.96 161.6)
 		(width 0.3)
-		(layer "F.Cu")
+		(layer "B.Cu")
 		(net 23)
 	)

Commit message: Se corrigio la Vista3DInferior
Parts:
- removed the G*** at (163.0, 144.6)
- added G***: LOGO, DibujoT:capibara3, B.Cu at (156.4, 150.5)
